File: schematic/schematic/schematic.kicad_sch (KiCad schematic)
At the start: 4 parts, among them J1 Conn_01x05, U1 74AHCT125

Commit message: finished the PCB and added the images
Parts:
- added C2: nF100, Capacitor_THT:C_Disc_D5.1mm_W3.2mm_P5.00mm, symbol Device:C
- added unit 4 of U1
- C1: value C -> uF10; footprint Capacitor_SMD:C_0805_2012Metric -> Capacitor_THT:C_Disc_D5.1mm_W3.2mm_P5.00mm
- U1: footprint (none) -> Package_DIP:DIP-14_W7.62mm
Connections:
- net +5V: now also C2.1, U1.13
- net GND: now also C2.2, U1.12
- net PICO_CLK: now also A1.29 (GPIO22); no longer A1.22 (GPIO17)
- net PICO_CS: now also A1.26 (GPIO20); no longer A1.24 (GPIO18)
- net PICO_DIN: now also A1.32 (GPIO27_ADC1); no longer A1.21 (GPIO16)
- no-connect marks 29 -> 30
Other:
- moved on the sheet: U1E
